File: kicad/elepajaradio.kicad_pcb (KiCad board)
At the start: 2 copper layers, 44 x 47 mm, 32 parts, among them J1 SPI, J2 UART, J3 vdd_gnd, J4 reset, J5 OLED, SW1 RotaryEncoder, SW2 SW_Push, SW3 SW_Push, U1 MAX2606, U3 ATmega328PB-A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

Commit message: pcb fix
Routing:
- net GND: track 7.79 -> 7.38 mm, vias 34 -> 39
Changed lines of the file:
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@@
   (segment (start 141.395 79.82) (end 139.6325 79.82) (width 0.25) (layer "F.Cu") (net 2))
   (segment (start 147.73 97.55) (end 149.45 97.55) (width 0.25) (layer "F.Cu") (net 2))
+  (segment (start 149.45 97.55) (end 149.75 97.25) (width 0.25) (layer "F.Cu") (net 2))
   (segment (start 139.23 98.35) (end 137.65 98.35) (width 0.25) (layer "F.Cu") (net 2))
   (segment (start 143.8 87.95) (end 143.25 88.5) (width 0.25) (layer "F.Cu") (net 2))
@@
   (via (at 155.25 105.25) (size 0.8) (drill 0.4) (layers "F.Cu" "B.Cu") (free) (net 2))
   (via (at 135.25 93.75) (size 0.8) (drill 0.4) (layers "F.Cu" "B.Cu") (free) (net 2))
+  (via (at 127.75 89.25) (size 0.8) (drill 0.4) (layers "F.Cu" "B.Cu") (free) (net 2))
   (via (at 154 107.75) (size 0.8) (drill 0.4) (layers "F.Cu" "B.Cu") (free) (net 2))
+  (via (at 131 77) (size 0.8) (drill 0.4) (layers "F.Cu" "B.Cu") (free) (net 2))
+  (via (at 131 78.25) (size 0.8) (drill 0.4) (layers "F.Cu" "B.Cu") (free) (net 2))
   (via (at 156 98.5) (size 0.8) (drill 0.4) (layers "F.Cu" "B.Cu") (free) (net 2))
   (via (at 152.75 105.25) (size 0.8) (drill 0.4) (layers "F.Cu" "B.Cu") (free) (net 2))
@@
   (via (at 135.25 92.25) (size 0.8) (drill 0.4) (layers "F.Cu" "B.Cu") (free) (net 2))
   (via (at 154 105.25) (size 0.8) (drill 0.4) (layers "F.Cu" "B.Cu") (free) (net 2))
+  (via (at 149.75 97.25) (size 0.8) (drill 0.4) (layers "F.Cu" "B.Cu") (net 2))
   (via (at 156 96) (size 0.8) (drill 0.4) (layers "F.Cu" "B.Cu") (free) (net 2))
   (via (at 136.5 89.25) (size 0.8) (drill 0.4) (layers "F.Cu" "B.Cu") (free) (net 2))
@@
   (via (at 156.5 105.25) (size 0.8) (drill 0.4) (layers "F.Cu" "B.Cu") (free) (net 2))
   (via (at 136.5 92.25) (size 0.8) (drill 0.4) (layers "F.Cu" "B.Cu") (free) (net 2))
+  (via (at 127.75 92.5) (size 0.8) (drill 0.4) (layers "F.Cu" "B.Cu") (free) (net 2))
   (via (at 156 94.75) (size 0.8) (drill 0.4) (layers "F.Cu" "B.Cu") (free) (net 2))
-  (segment (start 137.587299 98.412701) (end 137 99) (width 0.25) (layer "B.Cu") (net 2))
   (segment (start 128.15 100.825) (end 129.78 99.195) (width 0.25) (layer "F.Cu") (net 3))
   (segment (start 128.15 104.45) (end 128.15 100.825) (width 0.25) (layer "F.Cu") (net 3))

Commit message: fixes
Connections:
- AE1 pad 2: (no net) -> GND
Routing:
- net GND: vias 39 -> 41
Changed lines of the file:
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@@
     (pad "1" thru_hole roundrect (at 0 0 270) (size 2.3 2.3) (drill 1.5) (layers "*.Cu" "*.Mask") (remove_unused_layers) (keep_end_layers) (zone_layer_connections) (roundrect_rratio 0.087)
       (net 8 "Net-(AE1-A)") (pinfunction "A") (pintype "input"))
-    (pad "2" thru_hole circle (at -2.54 -2.54 270) (size 2.5 2.5) (drill 1.7) (layers "*.Cu" "*.Mask") (remove_unused_layers) (keep_end_layers) (zone_layer_connections))
-    (pad "2" thru_hole circle (at -2.54 2.54 270) (size 2.5 2.5) (drill 1.7) (layers "*.Cu" "*.Mask") (remove_unused_layers) (keep_end_layers) (zone_layer_connections))
-    (pad "2" thru_hole circle (at 2.54 -2.54 270) (size 2.5 2.5) (drill 1.7) (layers "*.Cu" "*.Mask") (remove_unused_layers) (keep_end_layers) (zone_layer_connections))
-    (pad "2" thru_hole circle (at 2.54 2.54 270) (size 2.5 2.5) (drill 1.7) (layers "*.Cu" "*.Mask") (remove_unused_layers) (keep_end_layers) (zone_layer_connections))
+    (pad "2" thru_hole circle (at -2.54 -2.54 270) (size 2.5 2.5) (drill 1.7) (layers "*.Cu" "*.Mask") (remove_unused_layers) (keep_end_layers) (zone_layer_connections)
+      (net 2 "GND"))
+    (pad "2" thru_hole circle (at -2.54 2.54 270) (size 2.5 2.5) (drill 1.7) (layers "*.Cu" "*.Mask") (remove_unused_layers) (keep_end_layers) (zone_layer_connections)
+      (net 2 "GND"))
+    (pad "2" thru_hole circle (at 2.54 -2.54 270) (size 2.5 2.5) (drill 1.7) (layers "*.Cu" "*.Mask") (remove_unused_layers) (keep_end_layers) (zone_layer_connections)
+      (net 2 "GND"))
+    (pad "2" thru_hole circle (at 2.54 2.54 270) (size 2.5 2.5) (drill 1.7) (layers "*.Cu" "*.Mask") (remove_unused_layers) (keep_end_layers) (zone_layer_connections)
+      (net 2 "GND"))
     (model "${KICAD6_3DMODEL_DIR}/Connector_Coaxial.3dshapes/SMA_Amphenol_901-143_Horizontal.wrl"
       (offset (xyz 0 0 0))
@@
   (via (at 157.25 96) (size 0.8) (drill 0.4) (layers "F.Cu" "B.Cu") (free) (net 2))
   (via (at 157.25 94.75) (size 0.8) (drill 0.4) (layers "F.Cu" "B.Cu") (free) (net 2))
+  (via (at 127.75 93.75) (size 0.8) (drill 0.4) (layers "F.Cu" "B.Cu") (free) (net 2))
   (via (at 157.25 97.25) (size 0.8) (drill 0.4) (layers "F.Cu" "B.Cu") (free) (net 2))
   (via (at 157.25 98.5) (size 0.8) (drill 0.4) (layers "F.Cu" "B.Cu") (free) (net 2))
+  (via (at 127.75 90.75) (size 0.8) (drill 0.4) (layers "F.Cu" "B.Cu") (free) (net 2))
   (via (at 135.25 90.75) (size 0.8) (drill 0.4) (layers "F.Cu" "B.Cu") (free) (net 2))
   (via (at 157.75 105.25) (size 0.8) (drill 0.4) (layers "F.Cu" "B.Cu") (free) (net 2))
@@
   (via (at 136.5 93.75) (size 0.8) (drill 0.4) (layers "F.Cu" "B.Cu") (free) (net 2))
   (via (at 135.25 92.25) (size 0.8) (drill 0.4) (layers "F.Cu" "B.Cu") (free) (net 2))
+  (via (at 127.75 92.25) (size 0.8) (drill 0.4) (layers "F.Cu" "B.Cu") (free) (net 2))
   (via (at 154 105.25) (size 0.8) (drill 0.4) (layers "F.Cu" "B.Cu") (free) (net 2))
   (via (at 149.75 97.25) (size 0.8) (drill 0.4) (layers "F.Cu" "B.Cu") (net 2))
@@
   (via (at 156.5 105.25) (size 0.8) (drill 0.4) (layers "F.Cu" "B.Cu") (free) (net 2))
   (via (at 136.5 92.25) (size 0.8) (drill 0.4) (layers "F.Cu" "B.Cu") (free) (net 2))
-  (via (at 127.75 92.5) (size 0.8) (drill 0.4) (layers "F.Cu" "B.Cu") (free) (net 2))
   (via (at 156 94.75) (size 0.8) (drill 0.4) (layers "F.Cu" "B.Cu") (free) (net 2))
   (segment (start 128.15 100.825) (end 129.78 99.195) (width 0.25) (layer "F.Cu") (net 3))
